Commit message: Add files via upload

File: urdf/3.urdf (robot description, URDF)
Before this commit: robot bot, 9 links, 8 joints
Links:
- added link imu; collision box size=0.027 0.02 0.004; visual box size=0.027 0.02 0.004
Joints:
- added joint base_link_to_imu_link: type fixed, parent base_link, child imu, origin xyz=-0.1125 -0.095 0.165 rpy=0.0 0.0 0.0, axis 0.0 1 0.0
